File: adb-usb-converter.kicad_pcb (KiCad board)
At the start: 2 copper layers, 44.7 x 17.8 mm, 3 parts, among them J1 Conn_01x05_Female, U1 ProMicro

Commit message: Forked by JK
Other:
- net class Default removed
- board text added: "ADB to USB adapter Forked by JK"
- board text added: "CODESQUAD JK"
- board text removed: "ADB to USB adapter by Ronan Gaillard rev A."
- board text removed: "JLCJLCJLCJLC"
